File: Conversor Boost-MCC. André, Nicollas e Vinicius/Conversor Boost-MCC. André, Nicollas e Vinicius.kicad_pcb (KiCad board)
At the start: 2 copper layers, 96 x 41 mm, 18 parts, among them J1 KRE KF128, J2 KRE KF128, J3 KRE KF128, Q1 IRF640, Q2 2N2907A, Q3 2N2222A, U1 UC3524

Commit message: Arquivos Gerbers gerados
Parts:
- Q2, Q3: footprint Package_TO_SOT_THT:TO-92 -> Package_TO_SOT_THT:TO-92_Inline_Wide
- moved NT1 35.5 mm to (103.5, 21.5)
- moved J3 34.6 mm to (65.5, 23.0), turned to 0 degrees
- moved C1 27.6 mm to (84.0, 28.4)
- moved C2 25.0 mm to (94.0, 28.4)
- moved L1 15.1 mm to (53.0, 44.2), turned to 180 degrees
- moved Q1 10.8 mm to (90.5, 41.0), turned to 180 degrees
- moved D1 9.85 mm to (86.0, 35.0)
- moved J1 6.73 mm to (52.5, 23.0), turned to 0 degrees
- moved Q3 6.07 mm to (109.7, 32.5), turned to 180 degrees
- moved Q2 5.58 mm to (109.6, 26.0), turned to 180 degrees
- moved C3 4.50 mm to (129.4, 30.5)
- moved J2 4.50 mm to (132.9, 53.0)
- moved R1 4.50 mm to (129.9, 34.4)
- moved R2 4.50 mm to (134.4, 44.6)
- moved R3 4.50 mm to (111.9, 47.7)
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Connections:
- L1 pad 1: +12V -> /Dreno
- L1 pad 2: /Dreno -> +12V
Routing:
- net GND: track 61.7 -> 11.5 mm
- net +12V: track 40.8 -> 11.6 mm
- net GNDPWR: track 27.9 -> 0.00 mm
- net +24V: track 67.9 -> 41.7 mm
- net +15V: track 57.9 -> 50.2 mm
- net Net-(Q2-B): track 21.0 -> 26.6 mm
- net /Dreno: track 35.5 -> 33.9 mm
- removed copper zone on F.Cu, net GND
- removed copper zone on F.Cu, net GNDPWR
Other:
- board size 96 x 41 mm -> 103.5 x 41 mm
