File: Conversor Boost-MCC. André, Nicollas e Vinicius/Conversor Boost-MCC. André, Nicollas e Vinicius.kicad_sch (KiCad schematic)
At the start: 17 parts, among them J1 KRE KF128, J2 KRE KF128, J3 KRE KF128, Q1 IRF640, Q2 2N2907A, Q3 2N2222A, U1 UC3524

Commit message: Layout finalizado
Parts:
- added NT1: NetTie_2, NetTie:NetTie-2_SMD_Pad2.0mm, symbol Device:NetTie_2
- L1: footprint (none) -> Indutores_Potência:Indutor_Potência
- Q1: footprint digikey-footprints:TO-220-3 -> Indutores_Potência:TO-220
- R2: footprint Resistor_THT:R_Axial_DIN0309_L9.0mm_D3.2mm_P2.54mm_Vertical -> Resistor_THT:R_Axial_DIN0207_L6.3mm_D2.5mm_P10.16mm_Horizontal
Connections:
- net GND: now also NT1.1; no longer C1.2, C2.2, J1.2 (Pin_2), J3.2 (Pin_2), Q1.3 (S)
- net Dreno: now reaches D1.2 (A), L1.2, Q1.1 (D)
- new net GNDPWR: C1.2, C2.2, J1.2 (Pin_2), J3.2 (Pin_2), NT1.2, Q1.3 (S)
Changed lines of the file:
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@@
+	(wire
+		(pts
+			(xy 134.62 60.96) (xy 137.16 60.96)
+		)
+		(stroke
+			(width 0)
+			(type default)
+		)
+	)
+	(wire
+		(pts
+			(xy 128.27 60.96) (xy 129.54 60.96)
+		)
+		(stroke
+			(width 0)
+			(type default)
+		)
+	)
 	(wire
 		(pts
@@
 	(wire
 		(pts
-			(xy 128.27 63.5) (xy 137.16 63.5)
-		)
-		(stroke
-			(width 0)
-			(type default)
-		)
-	)
-	(wire
-		(pts
 			(xy 140.97 34.29) (xy 143.51 34.29)
 		)
@@
 	(wire
 		(pts
-			(xy 128.27 66.04) (xy 128.27 63.5)
-		)
-		(stroke
-			(width 0)
-			(type default)
-		)
-	)
-	(wire
-		(pts
 			(xy 27.94 31.75) (xy 27.94 30.48)
 		)
@@
 	(wire
 		(pts
+			(xy 87.63 26.67) (xy 87.63 27.94)
+		)
+		(stroke
+			(width 0)
+			(type default)
+		)
+	)
+	(wire
+		(pts
 			(xy 101.6 77.47) (xy 101.6 83.82)
 		)
@@
 	(wire
 		(pts
-			(xy 137.16 63.5) (xy 137.16 66.04)
+			(xy 137.16 60.96) (xy 137.16 66.04)
 		)
 		(stroke
@@
 	(wire
 		(pts
+			(xy 128.27 60.96) (xy 128.27 66.04)
+		)
+		(stroke
+			(width 0)
+			(type default)
+		)
+	)
+	(wire
+		(pts
 			(xy 27.94 45.72) (xy 27.94 46.99)
 		)
@@
 			(width 0)
 			(type default)
+		)
+	)
+	(label "Dreno"
+		(at 87.63 26.67 90)
+		(effects
+			(font
+				(size 1.27 1.27)
+			)
+			(justify left bottom)
 		)
 	)
@@
 			)
 		)
-		(property "Footprint" "Resistor_THT:R_Axial_DIN0309_L9.0mm_D3.2mm_P2.54mm_Vertical"
+		(property "Footprint" "Resistor_THT:R_Axial_DIN0207_L6.3mm_D2.5mm_P10.16mm_Horizontal"
 			(at 26.416 100.584 90)
 			(effects
@@
 	)
 	(symbol
+		(lib_id "Device:NetTie_2")
+		(at 132.08 60.96 0)
+		(unit 1)
+		(exclude_from_sim no)
+		(in_bom no)
+		(on_board yes)
+		(dnp no)
+		(fields_autoplaced yes)
+		(property "Reference" "NT1"
+			(at 132.08 55.88 0)
+			(effects
+				(font
+					(size 1.27 1.27)
+				)
+			)
+		)
+		(property "Value" "NetTie_2"
+			(at 132.08 58.42 0)
+			(effects
+				(font
+					(size 1.27 1.27)
+				)
+			)
+		)
+		(property "Footprint" "NetTie:NetTie-2_SMD_Pad2.0mm"
+			(at 132.08 60.96 0)
+			(effects
+				(font
+					(size 1.27 1.27)
+				)
+				(hide yes)
+			)
+		)
+		(property "Datasheet" "~"
+			(at 132.08 60.96 0)
+			(effects
+				(font
+					(size 1.27 1.27)
+				)
+				(hide yes)
+			)
+		)
+		(property "Description" "Net tie, 2 pins"
+			(at 132.08 60.96 0)
+			(effects
+				(font
+					(size 1.27 1.27)
+				)
+				(hide yes)
+			)
+		)
+		(pin "2"
+		)
+		(pin "1"
+		)
+		(instances
+			(project ""
+				(path "/b343dbd4-cc43-4b9e-a40b-dc88b32413a9"
+					(reference "NT1")
+					(unit 1)
+				)
+			)
+		)
+	)
+	(symbol
 		(lib_id "power:+15V")
 		(at 110.49 71.12 0)
@@
 			)
 		)
-		(property "Footprint" ""
+		(property "Footprint" "Indutores_Potência:Indutor_Potência"
 			(at 77.47 27.94 0)
 			(effects
@@
 			)
 		)
-		(property "Footprint" "digikey-footprints:TO-220-3"
+		(property "Footprint" "Indutores_Potência:TO-220"
 			(at 90.17 33.02 0)
 			(effects
@@
 			)
 		)
-		(property "Sim.Pins" "1=D 2=G 3=S"
+		(property "Sim.Pins" "1=G 2=D 3=S"
 			(at 85.09 50.8 0)
 			(effects

Commit message: Arquivos Gerbers gerados
Parts:
- Q2, Q3: footprint Package_TO_SOT_THT:TO-92 -> Package_TO_SOT_THT:TO-92_Inline_Wide
Connections:
- net +12V: now also L1.2; no longer L1.1
- net Dreno: now also L1.1; no longer L1.2
Other:
- moved on the sheet: L1
Changed lines of the file:
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@@
 			)
 		)
-		(property "Footprint" "Package_TO_SOT_THT:TO-92"
+		(property "Footprint" "Package_TO_SOT_THT:TO-92_Inline_Wide"
 			(at 171.45 77.47 0)
 			(effects
@@
 	(symbol
 		(lib_id "Device:L")
-		(at 77.47 27.94 90)
+		(at 77.47 27.94 270)
 		(unit 1)
 		(exclude_from_sim no)
@@
 			)
 		)
-		(property "Footprint" "Package_TO_SOT_THT:TO-92"
+		(property "Footprint" "Package_TO_SOT_THT:TO-92_Inline_Wide"
 			(at 143.51 90.17 0)
 			(effects
